File: PCB Files/Squid60.sch (KiCad schematic (older format))
At the start: 19 parts, among them SW1 SW_Push, U1 ATmega32U4-AU, U2 PRTR5V0U2X, Y1 16Mhz

Commit message: Organization and images
Connections:
- net COL14: now reaches U1.32 (PC7)
Changed lines of the file:
@@
 	8000 10500 8450 10500
 $Sheet
-S 1800 1100 4350 2300
+S 1650 6100 4350 2300
 U 5EA8C563
 F0 "Matrix.sch" 50
@@
 Text GLabel 9050 9900 2    60   Input ~ 0
 COL0
+Text GLabel 9050 8200 2    60   Input ~ 0
+COL14
 $EndSCHEMATC

Commit message: Silkscreens
Parts:
- SW1: footprint Connector_PinSocket_2.00mm:PinSocket_1x02_P2.00mm_Horizontal -> Connector_PinSocket_2.00mm:PinSocket_1x02_P2.00mm_Vertical
Changed lines of the file:
@@
 F 0 "SW1" H 7200 7485 50  0000 C CNN
 F 1 "SW_Push" H 7200 7394 50  0000 C CNN
-F 2 "Connector_PinSocket_2.00mm:PinSocket_1x02_P2.00mm_Horizontal" H 7200 7400 50  0001 C CNN
+F 2 "Connector_PinSocket_2.00mm:PinSocket_1x02_P2.00mm_Vertical" H 7200 7400 50  0001 C CNN
 F 3 "" H 7200 7400 50  0001 C CNN
 	1    7200 7200
