File: PCB Files/Squid60.kicad_pcb (KiCad board)
At the start: 2 copper layers, 285 x 95.1 mm, 144 parts, among them SW1 SW_Push, U1 ATmega32U4-AU, U2 PRTR5V0U2X, Y1 16Mhz

Commit message: Silkscreens
Parts:
- removed REF**: 60_Outline, locallib:60_Outline-Modded
- added G***: LOGO, silks:SquidSilk, B.Cu at (185.3, 94.5)
- added G***: LOGO, silks:SquidSilk2, B.Cu at (118.1, 98.0)
- SW1: footprint Connector_PinSocket_2.00mm:PinSocket_1x02_P2.00mm_Horizontal -> Connector_PinSocket_2.00mm:PinSocket_1x02_P2.00mm_Vertical
- moved R1 0.18 mm to (53.1, 77.8)
- moved SW1 0.16 mm to (53.8, 75.7)
Routing:
- net +5V: track 130.4 -> 129.8 mm
Other:
- board outline removed
- board text added: "Designed by Alas"

Commit message: Couple Fixes
row 3 wasn't routed, row 1 had not been finished
Parts:
- moved R2 0.92 mm to (41.4, 92.0)
- moved C1 0.86 mm to (62.8, 80.0)
- moved C2 0.86 mm to (56.3, 80.1)
- moved Y1 0.86 mm to (59.6, 80.1)
- moved C6 0.50 mm to (39.4, 89.3)
- moved C5 0.20 mm to (49.6, 74.7)
Routing:
- net ROW3: track 59.7 -> 272.4 mm
- net ROW1: track 192.6 -> 220.1 mm, vias 0 -> 2
- net GND: track 49.5 -> 45.3 mm, vias 2 -> 1
- net +5V: track 129.8 -> 131.1 mm
- net Net-(C2-Pad1): track 8.32 -> 9.18 mm
- net Net-(C1-Pad1): track 11.6 -> 12.5 mm

Commit message: Removed Silkscreens
Because I don't to get sued

Also redid gerbers for that because again, yikes
Parts:
- removed G***: LOGO, silks:SquidSilk
- removed G***: LOGO, silks:SquidSilk2
Changed lines of the file:
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@@
   (general
     (thickness 1.6)
-    (drawings 1)
+    (drawings 2)
     (tracks 730)
     (zones 0)
-    (modules 145)
+    (modules 143)
     (nets 105)
   )
@@
     (add_net VCC)
   )
-  (module silks:SquidSilk (layer B.Cu)
-    (at 185.3184 94.488 180)
-    (fp_text reference G*** (at 0 0) (layer B.SilkS) hide
-      (effects (font (size 1.524 1.524) (thickness 0.3)) (justify mirror))
-    )
-    (fp_text value LOGO (at 0.75 0) (layer B.SilkS) hide
-      (effects (font (size 1.524 1.524) (thickness 0.3)) (justify mirror))
-    )
-    (fp_poly (pts (xy 8.819445 8.819444) (xy 13.229167 8.819444) (xy 13.229167 4.409722) (xy 17.638889 4.409722)
-      (xy 17.638889 0) (xy 22.048611 0) (xy 22.048611 -13.229167) (xy 17.638889 -13.229167)
-      (xy 17.638889 -4.409723) (xy 13.229167 -4.409723) (xy 13.229167 -13.229167) (xy 8.819445 -13.229167)
-      (xy 8.819445 -8.819445) (xy -13.229166 -8.819445) (xy -13.229166 -13.229167) (xy -17.638889 -13.229167)
-      (xy -17.638889 -4.409723) (xy -22.048611 -4.409723) (xy -22.048611 -13.229167) (xy -26.458333 -13.229167)
-      (xy -26.458333 0) (xy -22.048611 0) (xy -22.048611 4.409722) (xy -17.638889 4.409722)
-      (xy -13.229166 4.409722) (xy -13.229166 0) (xy -8.819444 0) (xy -8.819444 4.409722)
-      (xy 4.409723 4.409722) (xy 4.409723 0) (xy 8.819445 0) (xy 8.819445 4.409722)
-      (xy 4.409723 4.409722) (xy -8.819444 4.409722) (xy -13.229166 4.409722) (xy -17.638889 4.409722)
-      (xy -17.638889 8.819444) (xy -13.229166 8.819444) (xy -13.229166 13.229166) (xy -8.819444 13.229166)
-      (xy -8.819444 8.819444) (xy 4.409723 8.819444) (xy 4.409723 13.229166) (xy 8.819445 13.229166)
-      (xy 8.819445 8.819444)) (layer B.SilkS) (width 0.01))
-    (fp_poly (pts (xy 8.819445 17.638889) (xy 13.229167 17.638889) (xy 13.229167 13.229166) (xy 8.819445 13.229166)
-      (xy 8.819445 17.638889)) (layer B.SilkS) (width 0.01))
-    (fp_poly (pts (xy 8.819445 -17.638889) (xy 0 -17.638889) (xy 0 -13.229167) (xy 8.819445 -13.229167)
-      (xy 8.819445 -17.638889)) (layer B.SilkS) (width 0.01))
-    (fp_poly (pts (xy -17.638889 13.229166) (xy -17.638889 17.638889) (xy -13.229166 17.638889) (xy -13.229166 13.229166)
-      (xy -17.638889 13.229166)) (layer B.SilkS) (width 0.01))
-    (fp_poly (pts (xy -4.409722 -13.229167) (xy -4.409722 -17.638889) (xy -13.229166 -17.638889) (xy -13.229166 -13.229167)
-      (xy -4.409722 -13.229167)) (layer B.SilkS) (width 0.01))
-  )
-  (module silks:SquidSilk2 (layer B.Cu)
-    (at 118.0592 98.044 180)
-    (fp_text reference G*** (at 0 0) (layer B.SilkS) hide
-      (effects (font (size 1.524 1.524) (thickness 0.3)) (justify mirror))
-    )
-    (fp_text value LOGO (at 0.75 0) (layer B.SilkS) hide
-      (effects (font (size 1.524 1.524) (thickness 0.3)) (justify mirror))
-    )
-    (fp_poly (pts (xy 8.89 7.112) (xy 12.446 7.112) (xy 12.446 3.556) (xy 16.002 3.556)
-      (xy 16.002 10.668) (xy 19.558 10.668) (xy 19.558 -3.556) (xy 16.002 -3.556)
-      (xy 16.002 -7.112) (xy 12.446 -7.112) (xy 12.446 -10.668) (xy 8.89 -10.668)
-      (xy 8.89 -7.112) (xy -8.89 -7.112) (xy -8.89 -10.668) (xy -12.446 -10.668)
-      (xy -12.446 -7.112) (xy -16.002 -7.112) (xy -16.002 -3.556) (xy -19.558 -3.556)
-      (xy -19.558 10.668) (xy -16.002 10.668) (xy -16.002 3.556) (xy -12.446 3.556)
-      (xy -8.89 3.556) (xy -8.89 0) (xy -5.334 0) (xy -5.334 3.556)
-      (xy 5.334 3.556) (xy 5.334 0) (xy 8.89 0) (xy 8.89 3.556)
-      (xy 5.334 3.556) (xy -5.334 3.556) (xy -8.89 3.556) (xy -12.446 3.556)
-      (xy -12.446 7.112) (xy -8.89 7.112) (xy -8.89 10.668) (xy -5.334 10.668)
-      (xy -5.334 7.112) (xy 5.334 7.112) (xy 5.334 10.668) (xy 8.89 10.668)
-      (xy 8.89 7.112)) (layer B.SilkS) (width 0.01))
-    (fp_poly (pts (xy 8.89 14.224) (xy 12.446 14.224) (xy 12.446 10.668) (xy 8.89 10.668)
-      (xy 8.89 14.224)) (layer B.SilkS) (width 0.01))
-    (fp_poly (pts (xy 16.002 -10.668) (xy 16.002 -14.224) (xy 12.446 -14.224) (xy 12.446 -10.668)
-      (xy 16.002 -10.668)) (layer B.SilkS) (width 0.01))
-    (fp_poly (pts (xy -12.446 10.668) (xy -12.446 14.224) (xy -8.89 14.224) (xy -8.89 10.668)
-      (xy -12.446 10.668)) (layer B.SilkS) (width 0.01))
-    (fp_poly (pts (xy -12.446 -14.224) (xy -16.002 -14.224) (xy -16.002 -10.668) (xy -12.446 -10.668)
-      (xy -12.446 -14.224)) (layer B.SilkS) (width 0.01))
-  )
   (module Connector_PinSocket_2.00mm:PinSocket_1x02_P2.00mm_Vertical (layer F.Cu)
     (at 53.7784 75.692 90)
@@
     )
   )
-  (gr_text "Designed by Alas" (at 91.948 111.6076) (layer B.SilkS)
-    (effects (font (size 1 1) (thickness 0.15)) (justify mirror))
+  (gr_text "Designed by Alas" (at 105.5751 107.9246) (layer F.SilkS)
+    (effects (font (size 3 3) (thickness 0.5)))
+  )
+  (gr_text "Designed by Alas" (at 105.5751 107.6833) (layer B.SilkS)
+    (effects (font (size 3 3) (thickness 0.5)) (justify mirror))
   )
   (via (at 32.3596 36.4998) (size 0.8) (drill 0.4) (layers F.Cu B.Cu) (net 1))

Commit message: Ignore previous commit
I'm dumb, THIS commit fixes those things
Parts:
- added REF**: 60_Outline, locallib:60_Outline-Modded, F.Cu at (150.8, 65.9)
Other:
- board outline added: 285 x 95.1 mm
Changed lines of the file:
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@@
     (tracks 730)
     (zones 0)
-    (modules 143)
+    (modules 144)
     (nets 105)
   )
@@
     (add_net VCC)
   )
+  (module locallib:60_Outline-Modded (layer F.Cu)
+    (at 150.8125 65.88125)
+    (fp_text reference REF** (at -139 50.5) (layer Edge.Cuts) hide
+      (effects (font (size 1 1) (thickness 0.15)))
+    )
+    (fp_text value 60_Outline (at -139 49) (layer F.Fab) hide
+      (effects (font (size 1 1) (thickness 0.15)))
+    )
+    (fp_line (start -124.3 -48.9) (end -124.3 -45.75) (layer Dwgs.User) (width 0.15))
+    (fp_line (start -140.5 -47.3) (end -130.3 -47.3) (layer Edge.Cuts) (width 0.3))
+    (fp_arc (start -118.3 -47.8) (end -118.3 -47.3) (angle 90) (layer Edge.Cuts) (width 0.3))
+    (fp_arc (start -130.3 -47.8) (end -129.8 -47.8) (angle 90) (layer Edge.Cuts) (width 0.3))
+    (fp_line (start -129.8 -47.8) (end -118.8 -47.8) (layer Edge.Cuts) (width 0.3))
+    (fp_line (start 138.7 6.54905) (end 142.5 6.54905) (layer F.Mask) (width 2.5019))
+    (fp_line (start 138.7 6.54905) (end 142.5 6.54905) (layer B.Mask) (width 2.5019))
+    (fp_arc (start 138.7 9.2) (end 138.7 6.54905) (angle -90) (layer B.Mask) (width 2.5019))
+    (fp_arc (start 138.7 9.2) (end 138.7 6.54905) (angle -90) (layer F.Mask) (width 2.5019))
+    (fp_arc (start 138.7 9.2) (end 136.04905 9.2) (angle -90) (layer B.Mask) (width 2.5019))
+    (fp_arc (start 138.7 9.2) (end 136.04905 9.2) (angle -90) (layer F.Mask) (width 2.5019))
+    (fp_line (start 138.7 11.85095) (end 142.55 11.85095) (layer F.Mask) (width 2.5019))
+    (fp_line (start 138.7 11.85095) (end 142.55 11.85095) (layer B.Mask) (width 2.5019))
+    (fp_line (start -142.5 6.54905) (end -138.7 6.54905) (layer B.Mask) (width 2.5019))
+    (fp_line (start -142.5 6.54905) (end -138.7 6.54905) (layer F.Mask) (width 2.5019))
+    (fp_arc (start -138.7 9.2) (end -138.7 6.54905) (angle 90) (layer B.Mask) (width 2.5019))
+    (fp_arc (start -138.7 9.2) (end -138.7 6.54905) (angle 90) (layer F.Mask) (width 2.5019))
+    (fp_arc (start -138.7 9.2) (end -136.04905 9.2) (angle 90) (layer F.Mask) (width 2.5019))
+    (fp_arc (start -138.7 9.2) (end -136.04905 9.2) (angle 90) (layer B.Mask) (width 2.5019))
+    (fp_line (start -142.5 11.85095) (end -138.7 11.85095) (layer B.Mask) (width 2.5019))
+    (fp_line (start -142.5 11.85095) (end -138.7 11.85095) (layer F.Mask) (width 2.5019))
+    (fp_line (start 138.7 11.85095) (end 142.55 11.85095) (layer B.Cu) (width 2.5019))
+    (fp_line (start 138.7 6.54905) (end 142.5 6.54905) (layer F.Cu) (width 2.5019))
+    (fp_arc (start 138.7 9.2) (end 136.04905 9.2) (angle -90) (layer F.Cu) (width 2.5019))
+    (fp_arc (start 138.7 9.2) (end 138.7 6.54905) (angle -90) (layer F.Cu) (width 2.5019))
+    (fp_line (start 138.7 6.54905) (end 142.5 6.54905) (layer B.Cu) (width 2.5019))
+    (fp_line (start 138.7 11.85095) (end 142.55 11.85095) (layer F.Cu) (width 2.5019))
+    (fp_arc (start 138.7 9.2) (end 136.04905 9.2) (angle -90) (layer B.Cu) (width 2.5019))
+    (fp_arc (start 138.7 9.2) (end 138.7 6.54905) (angle -90) (layer B.Cu) (width 2.5019))
+    (fp_arc (start -138.7 9.2) (end -138.7 6.54905) (angle 90) (layer B.Cu) (width 2.5019))
+    (fp_arc (start -138.7 9.2) (end -136.04905 9.2) (angle 90) (layer B.Cu) (width 2.5019))
+    (fp_line (start -142.5 11.85095) (end -138.7 11.85095) (layer F.Cu) (width 2.5019))
+    (fp_line (start -142.5 11.85095) (end -138.7 11.85095) (layer B.Cu) (width 2.5019))
+    (fp_arc (start -138.7 9.2) (end -138.7 6.54905) (angle 90) (layer F.Cu) (width 2.5019))
+    (fp_arc (start -138.7 9.2) (end -136.04905 9.2) (angle 90) (layer F.Cu) (width 2.5019))
+    (fp_arc (start -138.7 9.2) (end -137.3 9.2) (angle 90) (layer Edge.Cuts) (width 0.3))
+    (fp_line (start -142.5 6.54905) (end -138.7 6.54905) (layer B.Cu) (width 2.5019))
+    (fp_line (start -142.5 6.54905) (end -138.7 6.54905) (layer F.Cu) (width 2.5019))
+    (fp_line (start 138.7 7.8) (end 142.5 7.8) (layer Edge.Cuts) (width 0.3))
+    (fp_line (start 138.7 10.6) (end 142.5 10.6) (layer Edge.Cuts) (width 0.3))
+    (fp_line (start 142.5 7.8) (end 142.5 -45.3) (layer Edge.Cuts) (width 0.3))
+    (fp_line (start 142.5 10.6) (end 142.5 45.3) (layer Edge.Cuts) (width 0.3))
+    (fp_arc (start 138.7 9.2) (end 137.3 9.2) (angle -90) (layer Edge.Cuts) (width 0.3))
+    (fp_arc (start 138.7 9.2) (end 138.7 7.8) (angle -90) (layer Edge.Cuts) (width 0.3))
+    (fp_line (start -142.5 7.8) (end -142.5 -45.3) (layer Edge.Cuts) (width 0.3))
+    (fp_line (start -138.7 7.8) (end -142.5 7.8) (layer Edge.Cuts) (width 0.3))
+    (fp_arc (start -138.7 9.2) (end -138.7 7.8) (angle 90) (layer Edge.Cuts) (width 0.3))
+    (fp_line (start -142.5 10.6) (end -138.7 10.6) (layer Edge.Cuts) (width 0.3))
+    (fp_line (start -142.5 45.3) (end -142.5 10.6) (layer Edge.Cuts) (width 0.3))
+    (fp_arc (start 140.5 -45.3) (end 140.5 -47.3) (angle 90) (layer Edge.Cuts) (width 0.3))
+    (fp_arc (start 140.5 45.3) (end 142.5 45.3) (angle 90) (layer Edge.Cuts) (width 0.3))
+    (fp_arc (start -140.5 45.3) (end -140.5 47.3) (angle 90) (layer Edge.Cuts) (width 0.3))
+    (fp_arc (start -140.5 -45.3) (end -142.5 -45.3) (angle 90) (layer Edge.Cuts) (width 0.3))
+    (fp_line (start 140.5 -47.3) (end -118.3 -47.3) (layer Edge.Cuts) (width 0.3))
+    (fp_line (start -140.5 47.3) (end 140.5 47.3) (layer Edge.Cuts) (width 0.3))
+    (pad 1 thru_hole circle (at -117.3 -19.4) (size 7.0013 7.0013) (drill 2.4994) (layers *.Cu *.Mask))
+    (pad 1 thru_hole circle (at -14.3 -0.3) (size 7.00024 7.00024) (drill oval 5.00126 2.49936) (layers *.Cu *.Mask))
+    (pad 1 thru_hole circle (at 48 37.9) (size 7.00024 7.00024) (drill oval 5.00126 2.49936) (layers *.Cu *.Mask))
+    (pad 1 thru_hole circle (at 117.55 -19.4) (size 7.00024 7.00024) (drill oval 5.00126 2.49936) (layers *.Cu *.Mask))
+    (pad 1 thru_hole circle (at -117.3 -21.7) (size 1 1) (drill 0.5) (layers *.Cu *.Mask))
+    (pad 1 thru_hole circle (at -119.6 -19.4) (size 1 1) (drill 0.5) (layers *.Cu *.Mask))
+    (pad 1 thru_hole circle (at -115 -19.4) (size 1 1) (drill 0.5) (layers *.Cu *.Mask))
+    (pad 1 thru_hole circle (at -117.3 -17.1) (size 1 1) (drill 0.5) (layers *.Cu *.Mask))
+    (pad 1 thru_hole circle (at -118.926346 -21.026346) (size 1 1) (drill 0.5) (layers *.Cu *.Mask))
+    (pad 1 thru_hole circle (at -115.673654 -21.026346) (size 1 1) (drill 0.5) (layers *.Cu *.Mask))
+    (pad 1 thru_hole circle (at -118.926346 -17.773654) (size 1 1) (drill 0.5) (layers *.Cu *.Mask))
+    (pad 1 thru_hole circle (at -115.673654 -17.773654) (size 1 1) (drill 0.5) (layers *.Cu *.Mask))
+    (pad 1 thru_hole circle (at 117.55 -21.7) (size 1 1) (drill 0.5) (layers *.Cu *.Mask))
+    (pad 1 thru_hole circle (at 117.55 -17.1) (size 1 1) (drill 0.5) (layers *.Cu *.Mask))
+    (pad 1 thru_hole circle (at 118.75 -17.1) (size 1 1) (drill 0.5) (layers *.Cu *.Mask))
+    (pad 1 thru_hole circle (at 116.35 -17.1) (size 1 1) (drill 0.5) (layers *.Cu *.Mask))
+    (pad 1 thru_hole circle (at 116.35 -21.7) (size 1 1) (drill 0.5) (layers *.Cu *.Mask))
+    (pad 1 thru_hole circle (at 118.75 -21.717) (size 1 1) (drill 0.5) (layers *.Cu *.Mask))
+    (pad 1 thru_hole circle (at 48 35.6) (size 1 1) (drill 0.5) (layers *.Cu *.Mask))
+    (pad 1 thru_hole circle (at 48 40.2) (size 1 1) (drill 0.5) (layers *.Cu *.Mask))
+    (pad 1 thru_hole circle (at 49.2 35.6) (size 1 1) (drill 0.5) (layers *.Cu *.Mask))
+    (pad 1 thru_hole circle (at 46.8 35.6) (size 1 1) (drill 0.5) (layers *.Cu *.Mask))
+    (pad 1 thru_hole circle (at 46.8 40.2) (size 1 1) (drill 0.5) (layers *.Cu *.Mask))
+    (pad 1 thru_hole circle (at 49.2 40.2) (size 1 1) (drill 0.5) (layers *.Cu *.Mask))
+    (pad 1 thru_hole circle (at -14.3 -2.6) (size 1 1) (drill 0.5) (layers *.Cu *.Mask))
+    (pad 1 thru_hole circle (at -13.1 -2.6) (size 1 1) (drill 0.5) (layers *.Cu *.Mask))
+    (pad 1 thru_hole circle (at -15.5 -2.6) (size 1 1) (drill 0.5) (layers *.Cu *.Mask))
+    (pad 1 thru_hole circle (at -14.3 2) (size 1 1) (drill 0.5) (layers *.Cu *.Mask))
+    (pad 1 thru_hole circle (at -15.5 2) (size 1 1) (drill 0.5) (layers *.Cu *.Mask))
+    (pad 1 thru_hole circle (at -13.1 2) (size 1 1) (drill 0.5) (layers *.Cu *.Mask))
+    (pad 1 thru_hole circle (at -136.1 9.2) (size 1 1) (drill 0.5) (layers *.Cu *.Mask))
+    (pad 1 thru_hole circle (at -138.7 6.6) (size 1 1) (drill 0.5) (layers *.Cu *.Mask))
+    (pad 1 thru_hole circle (at -138.7 11.8) (size 1 1) (drill 0.5) (layers *.Cu *.Mask))
+    (pad 1 thru_hole circle (at -136.861522 7.361522) (size 1 1) (drill 0.5) (layers *.Cu *.Mask))
+    (pad 1 thru_hole circle (at -136.861522 11.038478) (size 1 1) (drill 0.5) (layers *.Cu *.Mask))
+    (pad 1 thru_hole circle (at -140.742035 6.6) (size 1 1) (drill 0.5) (layers *.Cu *.Mask))
+    (pad 1 thru_hole circle (at -140.742035 11.8) (size 1 1) (drill 0.5) (layers *.Cu *.Mask))
+    (pad 1 thru_hole circle (at 136.1 9.2) (size 1 1) (drill 0.5) (layers *.Cu *.Mask))
+    (pad 1 thru_hole circle (at 136.861522 7.361522) (size 1 1) (drill 0.5) (layers *.Cu *.Mask))
+    (pad 1 thru_hole circle (at 138.7 6.6) (size 1 1) (drill 0.5) (layers *.Cu *.Mask))
+    (pad 1 thru_hole circle (at 140.742035 6.6) (size 1 1) (drill 0.5) (layers *.Cu *.Mask))
+    (pad 1 thru_hole circle (at 140.742035 11.8) (size 1 1) (drill 0.5) (layers *.Cu *.Mask))
+    (pad 1 thru_hole circle (at 138.7 11.8) (size 1 1) (drill 0.5) (layers *.Cu *.Mask))
+    (pad 1 thru_hole circle (at 136.861522 11.038478) (size 1 1) (drill 0.5) (layers *.Cu *.Mask))
+  )
   (module Connector_PinSocket_2.00mm:PinSocket_1x02_P2.00mm_Vertical (layer F.Cu)

Commit message: Fixed up the overlapping footprints and zipped gerbers
Parts:
- removed REF**: 60_Outline, locallib:60_Outline-Modded
- MX1, MX31: moved to B.Cu
- turned MX1 to 180 degrees
Connections:
- MX1 pad 2: Net-(D15-Pad2) -> Net-(D14-Pad2)
- MX31 pad 1: COL13 -> COL14
Routing:
- net Net-(D14-Pad2): track 22.5 -> 41.0 mm
- net Net-(D15-Pad2): track 46.2 -> 36.8 mm
- net Net-(D42-Pad2): track 52.2 -> 61.3 mm
- net COL13: track 320.3 -> 311.6 mm
- net COL14: track 347.9 -> 351.7 mm
Other:
- board outline removed
